Commit message: through task a.3, updated tasks file

File: nuturtle_description/urdf/turtlebot3_burger.urdf.xacro (robot description, xacro)
@@ -4,4 +4,7 @@
   xmlns:xacro="http://ros.org/wiki/xacro">
   <!-- <xacro:include filename="$(find turtlebot3_description)/urdf/common_properties.urdf"/> -->
+  <!-- load parameters from yaml file -->
+  <xacro:property name="yaml_file" value="$(find nuturtle_description)/config/diff_params.yaml" />
+  <xacro:property name="props" value="${xacro.load_yaml(yaml_file)['/**']['ros__parameters']}" />
   <!-- Init colour -->
   <material name="black">
@@ -52,5 +55,10 @@
       <origin xyz="-0.032 0 0.070" rpy="0 0 0"/>
       <geometry>
-        <box size="0.140 0.140 0.143"/>
+        <xacro:if value = "${props['collision_radius'] &lt; 0}">
+          <box size="0.140 0.140 0.143"/>
+        </xacro:if>
+        <xacro:unless value = "${props['collision_radius'] &lt; 0}">
+          <cylinder length="0.143" radius="${props['collision_radius']}"/>
+        </xacro:unless>
       </geometry>
     </collision>
@@ -64,5 +72,5 @@
     <parent link="base_link"/>
     <child link="wheel_left_link"/>
-    <origin xyz="0.0 0.08 0.023" rpy="-1.57 0 0"/>
+    <origin xyz="0.0 ${props['track_width']/2} 0.023" rpy="-1.57 0 0"/>
     <axis xyz="0 0 1"/>
   </joint>
@@ -78,5 +86,5 @@
       <origin xyz="0 0 0" rpy="0 0 0"/>
       <geometry>
-        <cylinder length="0.018" radius="0.033"/>
+        <cylinder length="0.018" radius="${props['wheel_radius']}"/>
       </geometry>
     </collision>
@@ -90,5 +98,5 @@
     <parent link="base_link"/>
     <child link="wheel_right_link"/>
-    <origin xyz="0.0 -0.080 0.023" rpy="-1.57 0 0"/>
+    <origin xyz="0.0 -${props['track_width']/2} 0.023" rpy="-1.57 0 0"/>
     <axis xyz="0 0 1"/>
   </joint>
@@ -104,5 +112,5 @@
       <origin xyz="0 0 0" rpy="0 0 0"/>
       <geometry>
-        <cylinder length="0.018" radius="0.033"/>
+        <cylinder length="0.018" radius="${props['wheel_radius']}"/>
       </geometry>
     </collision>

Commit message: progress in task a.4, color of the base link is changing according to launchfile argument

File: nuturtle_description/urdf/turtlebot3_burger.urdf.xacro (robot description, xacro)
@@ -7,4 +7,6 @@
   <xacro:property name="yaml_file" value="$(find nuturtle_description)/config/diff_params.yaml" />
   <xacro:property name="props" value="${xacro.load_yaml(yaml_file)['/**']['ros__parameters']}" />
+  <!-- arguments -->
+  <xacro:arg name="color" default="light_black"/>
   <!-- Init colour -->
   <material name="black">
@@ -38,4 +40,7 @@
     <color rgba="1.0 1.0 1.0 1.0"/>
   </material>
+  <material name="purple">
+    <color rgba="0.3 0.16 0.52 1.0"/>
+  </material>
   <link name="base_footprint"/>
   <joint name="base_joint" type="fixed">
@@ -50,5 +55,5 @@
         <mesh filename="package://nuturtle_description/meshes/burger_base.stl" scale="0.001 0.001 0.001"/>
       </geometry>
-      <material name="light_black"/>
+      <material name="$(arg color)"/>
     </visual>
     <collision>
